Commit message: Driving in Gazebo

File: description/robot_core.xacro (robot description, xacro)
@@ -39,4 +39,7 @@
         </xacro:inertial_box>
     </link>
+    <gazebo reference = "chassis">
+        <material>Gazebo/White</material>
+    </gazebo>
     <gazebo>
         <plugin name="joint_state_publisher" filename="libgazebo_ros_joint_state_publisher.so">
@@ -66,4 +69,7 @@
         </xacro:inertial_cylinder>
     </link>
+    <gazebo reference = "left_wheel">
+        <material>Gazebo/Blue</material>
+    </gazebo>
     <joint name = "right_wheel_joint" type="continuous">
         <parent link = "base_link"/>
@@ -88,4 +94,7 @@
         </xacro:inertial_cylinder>
     </link>
+    <gazebo reference = "right_wheel">
+        <material>Gazebo/Blue</material>
+    </gazebo>
     <joint name = "caster_wheel_joint" type = "fixed">
         <parent link = "chassis"/>
@@ -109,3 +118,8 @@
         </xacro:inertial_sphere>
     </link>
+    <gazebo reference = "caster_wheel">
+        <material>Gazebo/Black</material>
+        <mu1 value = "0.001"/>
+        <mu2 value = "0.001"/>
+    </gazebo>
 </robot>
